File: hardware/Kicad/Cape-485-BBB.sch (KiCad schematic (older format))
At the start: 29 parts, among them J1 RJ25, P1 CONN_01X01, SW1 Switch_DPST, SW2 Switch_DPST, U1 MAX3107E, U2 DCP010505, U3 IL3685, X1 OSCILADOR

Commit message: new hardware version
Parts:
- removed C1: 2u2, Capacitors_SMD:C_0805, symbol C_Small
- removed C2: 0.1u, Capacitors_SMD:C_0805, symbol C_Small
- removed JP1: Jumper_NO_Small, symbol Jumper_NO_Small
- removed P1: CONN_01X01, Symbols:Symbol_Danger_CopperTop_Small, symbol CONN_01X01
- removed R5, R6: 270r, Resistors_SMD:R_0805, symbol R
- removed R7: 120r, Resistors_SMD:R_0805, symbol R
- removed SW1, SW2: Switch_DPST, CapeBBB:Switch_2posicoes_SMD, symbol Switch_DPST
- removed U2: DCP010505, Housings_DIP:DIP-14__300, symbol DCP010505
- added C13: 0.1uF, Capacitors_SMD:C_0805, symbol C_Small
- added C14: 2.2uF, Capacitors_SMD:C_0805, symbol C_Small
- added C15: 1uF, Capacitors_SMD:C_0805, symbol C_Small
- added C16: 100n, Capacitors_SMD:C_0805, symbol C_Small
- added D2, D3, D4: LED, LEDs:LED_0805, symbol LED
- added J1: RJ25, CapeBBB:RJ25, symbol RJ25
- added JP3, JP4: Jumper_NO_Small, Measurement_Points:Test_Point, symbol Jumper_NO_Small
- added P10: CONN_02X05, Pin_Headers:Pin_Header_Straight_2x05, symbol CONN_02X05
- added Q1, Q2, Q3: BSR14, TO_SOT_Packages_SMD:SOT-23, symbol BC548
- added R10: 120r, Resistors_SMD:R_0805, symbol R
- added R11, R9: 1k, Resistors_SMD:R_0805, symbol R
- added R12, R14, R16: 10k, Resistors_SMD:R_0805, symbol R
- added R13, R15, R17: 100r, Resistors_SMD:R_0805, symbol R
- added R4, R8: 150r, Resistors_SMD:R_0805, symbol R
- added U4: DCR01XXXXU, Housings_SOIC:SOIC-28_7.5x17.9mm_Pitch1.27mm, symbol DCR01XXXXU
- added U5, U6: TS5A21366, symbol TS5A21366
- C10: value 47n -> 10u; symbol C_Small -> CP1_Small
- C11: value 10u -> 47n
- renumbered J1 to J2
Connections:
- net labels added: 1, 16, 2, 4, 8, LED1, LED2, LED3
- net labels removed: I1, I2, INPUT0, INPUT1, OK, OUTPUT
- wire segments 131 -> 162
- no-connect marks 79 -> 82
Other:
- note added: "Alimentação Isolada"
- note added: "ENDERECO\n(MODO SLAVE)"
- moved on the sheet: C11, C3, C4, C5, C6, C7, C8, C9, D1, J2, R2, R3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
